Commit message: update locomotion policy of g1 on warehouse

File: backend/assets/g1/g1_12dof.urdf (robot description, URDF)
Before this commit: robot g1_12dof, 31 links, 30 joints
Joints:
- joint left_elbow_joint: origin xyz=0.015783 0 -0.080518 rpy=0 0 0 -> xyz=0.015783 0 -0.080518 rpy=0 0.8 0
- joint left_hip_pitch_joint: limit lower=-2.5307 upper=2.8798 effort=88 velocity=32 -> lower=-1.0 upper=1.0 effort=88 velocity=32
- joint left_hip_roll_joint: limit lower=-0.5236 upper=2.9671 effort=139 velocity=20 -> lower=-0.2 upper=0.6 effort=139 velocity=20
- joint left_hip_yaw_joint: limit lower=-2.7576 upper=2.7576 effort=88 velocity=32 -> lower=-0.2 upper=0.2 effort=88 velocity=32
- joint right_elbow_joint: origin xyz=0.015783 0 -0.080518 rpy=0 0 0 -> xyz=0.015783 0 -0.080518 rpy=0 0.8 0
- joint right_hip_pitch_joint: limit lower=-2.5307 upper=2.8798 effort=88 velocity=32 -> lower=-1.0 upper=1.0 effort=88 velocity=32
- joint right_hip_roll_joint: limit lower=-2.9671 upper=0.5236 effort=139 velocity=20 -> lower=-0.6 upper=0.2 effort=139 velocity=20
- joint right_hip_yaw_joint: limit lower=-2.7576 upper=2.7576 effort=88 velocity=32 -> lower=-0.2 upper=0.2 effort=88 velocity=32
